Commit message: modified launch_mappingbot.launch.py

File: description/ros2_control.xacro (robot description, xacro)
@@ -1,5 +1,35 @@
 <?xml version="1.0"?>
 <robot xmlns:xacro="http://www.ros.org/wiki/xacro" >
-    <ros2_control name="GazeboSystem" type="system">
+    <ros2_control name="RealRobot" type="system">
+        <hardware>
+            <plugin>mappingbot_hardware/MappingbotHardware</plugin>
+            <param name="left_wheel_name">left_wheel_joint</param>
+            <param name="right_wheel_name">right_wheel_joint</param>
+            <param name="loop_rate">100</param>
+            <param name="serial_port">/dev/ttyAMA0</param>
+            <param name="baud_rate">115200</param>
+            <!-- <param name="timeout_ms"></param> -->
+            <!-- <param name="enc_counts_per_rev"></param> -->
+        </hardware>
+        <joint name="left_wheel_joint">
+            <command_interface name="velocity"/>
+                <!-- <param name="min">-10</param>
+                <param name="max">10</param> -->
+            <!-- </command_interface> -->
+            <state_interface name="velocity"/>
+            <state_interface name="position"/>
+            <param name="motor_id">1</param>
+        </joint>
+        <joint name="right_wheel_joint">
+            <command_interface name="velocity"/>
+                <!-- <param name="min">-10</param>
+                <param name="max">10</param> -->
+            <!-- </command_interface> -->
+            <state_interface name="velocity"/>
+            <state_interface name="position"/>
+            <param name="motor_id">2</param>
+        </joint>
+    </ros2_control>
+    <!-- <ros2_control name="GazeboSystem" type="system">
         <hardware>
             <plugin>gazebo_ros2_control/GazeboSystem</plugin>
@@ -21,5 +51,5 @@
             <state_interface name="position"/>
         </joint>
-    </ros2_control>
+    </ros2_control> -->
     <gazebo>
         <plugin name="diff_drive" filename="libgazebo_ros2_control.so">
