Commit message: adding slam and nav2

File: description/lidar.xacro (robot description, xacro)
@@ -4,5 +4,5 @@
         <parent link="chassis"/>
         <child link="laser_frame"/>
-        <origin xyz="0.1 0 0.15" rpy="0 0 0"/>
+        <origin xyz="-0.1 0 0.15" rpy="0 0 0"/>
     </joint>
     <link name="laser_frame">

File: description/robot.urdf.xacro (robot description, xacro)
@@ -2,4 +2,5 @@
 <robot xmlns:xacro="http://www.ros.org/wiki/xacro"  name="robot">
     <xacro:arg name="use_ros2_control" default="true"/>
+    <xacro:arg name="sim_mode" default="false"/>
     <xacro:include filename="robot_core.xacro" />
     <xacro:if value="$(arg use_ros2_control)">

File: description/robot_core.xacro (robot description, xacro)
@@ -36,13 +36,21 @@
     <link name="base_link">
     </link>
+    <!-- BASE FOOTPRINT LINK -->
+    <joint name="base_footprint_joint" type="fixed">
+        <parent link="base_link"/>
+        <child link="base_footprint"/>
+        <origin xyz="0 0 0" rpy="0 0 0 "/>
+    </joint>
+    <link name="base_footprint">
+    </link>
     <!-- CHASSIS LINK -->
     <joint name="chassis_joint" type="fixed">
         <parent link="base_link"/>
         <child link="chassis"/>
-        <origin xyz="-${wheel_offset_x} 0 -${wheel_offset_z}"/>
+        <origin xyz="${wheel_offset_x} 0 -${wheel_offset_z}"/>
     </joint>
     <link name="chassis">
         <visual>
-            <origin xyz = "${chassis_length/2} 0 ${chassis_height/2}"/>
+            <origin xyz = "-${chassis_length/2} 0 ${chassis_height/2}"/>
             <geometry>
                 <box size="${chassis_length} ${chassis_width} ${chassis_height}"/>
@@ -51,5 +59,5 @@
         </visual>
      <collision>
-            <origin xyz = "${chassis_length/2} 0 ${chassis_height/2}"/>
+            <origin xyz = "-${chassis_length/2} 0 ${chassis_height/2}"/>
             <geometry>
                 <box size="${chassis_length} ${chassis_width} ${chassis_height}"/>
@@ -57,5 +65,5 @@
         </collision>
         <xacro:inertial_box mass="${chassis_mass}" x="${chassis_length}" y="${chassis_width}" z="${chassis_height}">
-            <origin xyz="${chassis_length/2} 0 ${chassis_height/2}" rpy="0 0 0"/>
+            <origin xyz="-${chassis_length/2} 0 ${chassis_height/2}" rpy="0 0 0"/>
         </xacro:inertial_box>
     </link>
@@ -67,6 +75,6 @@
         <parent link="base_link"/>
         <child link="left_wheel"/>
-        <origin xyz="0 ${wheel_offset_y} 0" rpy="${pi/2} 0 0"/>
-        <axis xyz="0 0 -1"/>
+        <origin xyz="0 ${wheel_offset_y} 0" rpy="-${pi/2} 0 0"/>
+        <axis xyz="0 0 1"/>
     </joint>
     <link name="left_wheel">
@@ -93,6 +101,6 @@
         <parent link="base_link"/>
         <child link="right_wheel"/>
-        <origin xyz="0 -${wheel_offset_y} 0" rpy="-${pi/2} 0 0"/>
-        <axis xyz="0 0 1"/>
+        <origin xyz="0 -${wheel_offset_y} 0" rpy="${pi/2} 0 0"/>
+        <axis xyz="0 0 -1"/>
     </joint>
     <link name="right_wheel">
@@ -119,5 +127,5 @@
         <parent link="chassis"/>
         <child link="left_caster_wheel"/>
-        <origin xyz="${caster_wheel_offset_x} ${caster_wheel_offset_y} ${caster_wheel_offset_z}"/>
+        <origin xyz="-${caster_wheel_offset_x} ${caster_wheel_offset_y} ${caster_wheel_offset_z}"/>
     </joint>
     <link name="left_caster_wheel">
@@ -146,5 +154,5 @@
         <parent link="chassis"/>
         <child link="right_caster_wheel"/>
-        <origin xyz="${caster_wheel_offset_x} -${caster_wheel_offset_y} ${caster_wheel_offset_z}"/>
+        <origin xyz="-${caster_wheel_offset_x} -${caster_wheel_offset_y} ${caster_wheel_offset_z}"/>
     </joint>
     <link name="right_caster_wheel">

File: description/ros2_control.xacro (robot description, xacro)
@@ -1,55 +1,60 @@
 <?xml version="1.0"?>
 <robot xmlns:xacro="http://www.ros.org/wiki/xacro" >
-    <ros2_control name="RealRobot" type="system">
-        <hardware>
-            <plugin>hoverboard_driver/hoverboard_driver</plugin>
-            <param name="device">/dev/ttyAMA0</param>
-            <param name="wheel_radius">0.0825</param>
-            <param name="max_velocity">1.0</param>
-            <param name="baud_rate">115200</param>
-        </hardware>
-        <joint name="left_wheel_joint">
-            <command_interface name="velocity"/>
-                <!-- <param name="min">-10</param>
-                <param name="max">10</param> -->
-            <!-- </command_interface> -->
-            <state_interface name="position"/>
-            <state_interface name="velocity"/>
-            <param name="motor_id">1</param>
-        </joint>
-        <joint name="right_wheel_joint">
-            <command_interface name="velocity"/>
-                <!-- <param name="min">-10</param>
-                <param name="max">10</param> -->
-            <!-- </command_interface> -->
-            <state_interface name="position"/>
-            <state_interface name="velocity"/>
-            <param name="motor_id">2</param>
-        </joint>
-    </ros2_control>
-    <!-- <ros2_control name="GazeboSystem" type="system">
-        <hardware>
-            <plugin>gazebo_ros2_control/GazeboSystem</plugin>
-        </hardware>
-        <joint name="left_wheel_joint">
-            <command_interface name="velocity">
-                <param name="min">-10</param>
-                <param name="max">10</param>
-            </command_interface>
-            <state_interface name="velocity"/>
-            <state_interface name="position"/>
-        </joint>
-        <joint name="right_wheel_joint">
-            <command_interface name="velocity">
-                <param name="min">-10</param>
-                <param name="max">10</param>
-            </command_interface>
-            <state_interface name="velocity"/>
-            <state_interface name="position"/>
-        </joint>
-    </ros2_control> -->
+    <xacro:unless value="$(arg sim_mode)">
+        <ros2_control name="RealRobot" type="system">
+            <hardware>
+                <plugin>hoverboard_driver/hoverboard_driver</plugin>
+                <param name="device">/dev/ttyAMA0</param>
+                <param name="wheel_radius">0.0825</param>
+                <param name="max_velocity">1.0</param>
+                <param name="baud_rate">115200</param>
+            </hardware>
+            <joint name="left_wheel_joint">
+                <command_interface name="velocity"/>
+                    <!-- <param name="min">-10</param>
+                    <param name="max">10</param> -->
+                <!-- </command_interface> -->
+                <state_interface name="position"/>
+                <state_interface name="velocity"/>
+                <param name="motor_id">1</param>
+            </joint>
+            <joint name="right_wheel_joint">
+                <command_interface name="velocity"/>
+                    <!-- <param name="min">-10</param>
+                    <param name="max">10</param> -->
+                <!-- </command_interface> -->
+                <state_interface name="position"/>
+                <state_interface name="velocity"/>
+                <param name="motor_id">2</param>
+            </joint>
+        </ros2_control>
+    </xacro:unless>
+    <xacro:if value="$(arg sim_mode)">
+        <ros2_control name="GazeboSystem" type="system">
+            <hardware>
+                <plugin>gazebo_ros2_control/GazeboSystem</plugin>
+            </hardware>
+            <joint name="left_wheel_joint">
+                <command_interface name="velocity">
+                    <param name="min">-10</param>
+                    <param name="max">10</param>
+                </command_interface>
+                <state_interface name="velocity"/>
+                <state_interface name="position"/>
+            </joint>
+            <joint name="right_wheel_joint">
+                <command_interface name="velocity">
+                    <param name="min">-10</param>
+                    <param name="max">10</param>
+                </command_interface>
+                <state_interface name="velocity"/>
+                <state_interface name="position"/>
+            </joint>
+        </ros2_control>
+    </xacro:if>
     <gazebo>
-        <plugin name="diff_drive" filename="libgazebo_ros2_control.so">
+        <plugin name="gazebo_ros2_control" filename="libgazebo_ros2_control.so">
             <parameters>$(find mappingbot)/config/my_controllers.yaml</parameters>
+            <parameters>$(find mappingbot)/config/gaz_ros2_ctl_use_sim.yaml</parameters>
         </plugin>
     </gazebo>
