Commit message: Gazebo sim integration

File: description/robot_core.xacro (robot description, xacro)
@@ -57,4 +57,7 @@
         </xacro:inertial_box>
     </link>
+    <gazebo reference="chassis">
+        <material>Gazebo/White</material>
+    </gazebo>
     <!-- LEFT WHEEL LINK -->
     <joint name="left_wheel_joint" type="continuous">
@@ -80,4 +83,7 @@
         </xacro:inertial_cylinder>
     </link>
+    <gazebo reference="left_wheel">
+        <material>Gazebo/Blue</material>
+    </gazebo>
     <!-- RIGHT WHEEL LINK -->
     <joint name="right_wheel_joint" type="continuous">
@@ -103,4 +109,7 @@
         </xacro:inertial_cylinder>
     </link>
+    <gazebo reference="right_wheel">
+        <material>Gazebo/Blue</material>
+    </gazebo>
     <!-- LEFT CASTER WHEEL -->
     <joint name="left_caster_wheel_joint" type="fixed">
@@ -125,4 +134,9 @@
         </xacro:inertial_sphere>
     </link>
+    <gazebo reference="left_caster_wheel">
+        <material>Gazebo/Black</material>
+        <mu1 value="0.001"/>
+        <mu2 value="0.001"/>
+    </gazebo>
     <!-- RIGHT CASTER WHEEL -->
     <joint name="right_caster_wheel_joint" type="fixed">
@@ -147,3 +161,8 @@
         </xacro:inertial_sphere>
     </link>
+    <gazebo reference="right_caster_wheel">
+        <material>Gazebo/Black</material>
+        <mu1 value="0.001"/>
+        <mu2 value="0.001"/>
+    </gazebo>
 </robot>

Commit message: Get real robot working

File: description/robot_core.xacro (robot description, xacro)
@@ -67,6 +67,6 @@
         <parent link="base_link"/>
         <child link="left_wheel"/>
-        <origin xyz="0 ${wheel_offset_y} 0" rpy="-${pi/2} 0 0"/>
-        <axis xyz="0 0 1"/>
+        <origin xyz="0 ${wheel_offset_y} 0" rpy="${pi/2} 0 0"/>
+        <axis xyz="0 0 -1"/>
     </joint>
     <link name="left_wheel">
@@ -93,6 +93,6 @@
         <parent link="base_link"/>
         <child link="right_wheel"/>
-        <origin xyz="0 -${wheel_offset_y} 0" rpy="${pi/2} 0 0"/>
-        <axis xyz="0 0 -1"/>
+        <origin xyz="0 -${wheel_offset_y} 0" rpy="-${pi/2} 0 0"/>
+        <axis xyz="0 0 1"/>
     </joint>
     <link name="right_wheel">

File: description/ros2_control.xacro (robot description, xacro)
@@ -3,12 +3,9 @@
     <ros2_control name="RealRobot" type="system">
         <hardware>
-            <plugin>mappingbot_hardware/MappingbotHardware</plugin>
-            <param name="left_wheel_name">left_wheel_joint</param>
-            <param name="right_wheel_name">right_wheel_joint</param>
-            <param name="loop_rate">100</param>
-            <param name="serial_port">/dev/ttyAMA0</param>
+            <plugin>hoverboard_driver/hoverboard_driver</plugin>
+            <param name="device">/dev/ttyAMA0</param>
+            <param name="wheel_radius">0.0825</param>
+            <param name="max_velocity">1.0</param>
             <param name="baud_rate">115200</param>
-            <!-- <param name="timeout_ms"></param> -->
-            <!-- <param name="enc_counts_per_rev"></param> -->
         </hardware>
         <joint name="left_wheel_joint">
@@ -17,6 +14,6 @@
                 <param name="max">10</param> -->
             <!-- </command_interface> -->
+            <state_interface name="position"/>
             <state_interface name="velocity"/>
-            <state_interface name="position"/>
             <param name="motor_id">1</param>
         </joint>
@@ -26,6 +23,6 @@
                 <param name="max">10</param> -->
             <!-- </command_interface> -->
+            <state_interface name="position"/>
             <state_interface name="velocity"/>
-            <state_interface name="position"/>
             <param name="motor_id">2</param>
         </joint>

Commit message: get real robot working

File: description/robot_core.xacro (robot description, xacro)
@@ -68,5 +68,5 @@
         <child link="left_wheel"/>
         <origin xyz="0 ${wheel_offset_y} 0" rpy="${pi/2} 0 0"/>
-        <axis xyz="0 0 -1"/>
+        <axis xyz="0 0 1"/>
     </joint>
     <link name="left_wheel">
@@ -94,5 +94,5 @@
         <child link="right_wheel"/>
         <origin xyz="0 -${wheel_offset_y} 0" rpy="-${pi/2} 0 0"/>
-        <axis xyz="0 0 1"/>
+        <axis xyz="0 0 -1"/>
     </joint>
     <link name="right_wheel">

Commit message: get real robot working

File: description/robot_core.xacro (robot description, xacro)
@@ -68,5 +68,5 @@
         <child link="left_wheel"/>
         <origin xyz="0 ${wheel_offset_y} 0" rpy="${pi/2} 0 0"/>
-        <axis xyz="0 0 1"/>
+        <axis xyz="0 0 -1"/>
     </joint>
     <link name="left_wheel">
@@ -94,5 +94,5 @@
         <child link="right_wheel"/>
         <origin xyz="0 -${wheel_offset_y} 0" rpy="-${pi/2} 0 0"/>
-        <axis xyz="0 0 -1"/>
+        <axis xyz="0 0 1"/>
     </joint>
     <link name="right_wheel">

Commit message: adding slam and nav2

File: description/robot_core.xacro (robot description, xacro)
@@ -19,8 +19,8 @@
     <!-- ROBOT PARAMETERS -->
     <xacro:property name="wheel_radius" value="0.0825"/>
-    <xacro:property name="wheel_thickness" value="0.05"/>
+    <xacro:property name="wheel_thickness" value="0.04"/>
     <xacro:property name="wheel_mass" value="2.0"/>
     <xacro:property name="wheel_offset_x" value="0.1"/>
-    <xacro:property name="wheel_offset_y" value="0.25"/>
+    <xacro:property name="wheel_offset_y" value="0.19"/>
     <xacro:property name="wheel_offset_z" value="0.05"/>
     <xacro:property name="chassis_height" value="0.138"/>
