Commit message: pure_pursuit

File: description/gazebo_control.xacro (robot description, xacro)
@@ -6,5 +6,5 @@
             <left_joint>left_wheel_joint</left_joint>
             <right_joint>right_wheel_joint</right_joint>
-            <wheel_separation>0.5</wheel_separation>
+            <wheel_separation>0.38</wheel_separation>
             <wheel_diameter>0.165</wheel_diameter>
             <!-- LIMITS -->

File: description/lidar.xacro (robot description, xacro)
@@ -4,5 +4,5 @@
         <parent link="chassis"/>
         <child link="laser_frame"/>
-        <origin xyz="-0.1 0 0.15" rpy="0 0 0"/>
+        <origin xyz="-0.171 0 0.175" rpy="0 0 0"/>
     </joint>
     <link name="laser_frame">
